File: hardware/kicad/lfp8_ch2.kicad_sch (KiCad schematic)
At the start: 89 parts, among them J201 XH-6P, Q201 AO3401A, Q202 MMBT3904, Q203 2N7002, Q204 AO3400A, Q205 AO3400A, Q206 MMBT3904, Q207 MMBT3906, Q208 AO3400A, Q209 MMBT3906, Q210 MMBT3904, Q211 MMBT3904, U201 LM324

Commit message: Firmware: one IR pulse per scan sweep; researched JLCPCB cost estimate
- fix: IR measurements that became ready together ran back to back, each
  holding the ADC ~1.1 s, so the other channels went stale and faulted
  (FAULT_ADC). The scanner now starts at most one IR pulse per full sweep,
  round robin. New regression tests: 8 simultaneous IRs, and 3 IRs while
  5 channels discharge (78 host tests pass, ESP32-C3 build OK)
- parts: 7 resistor values are JLC 'preferred extended' (no loading fee),
  not basic; labels corrected, schematic regenerated (netlist unchanged)
- ORDERING_AND_ASSEMBLY: per-board cost table for 2 / 5 / 10 assembled boards
  from fee research, the JLC part database and 2026 checkout records

Co-Authored-By: Claude Opus 5.5 <noreply@anthropic.com>
Claude-Session: https://claude.ai/code/session_01741JMFwAZptriPav2AH4Eo
Parts:
- R220, R230, R231, R243, R255: JLC Basic -> Preferred
Changed lines of the file:
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@@
     (property "Datasheet" "~" (at 243.84 81.28 0) (effects (font (size 1.27 1.27)) hide))
     (property "LCSC" "C23146" (at 243.84 81.28 0) (effects (font (size 1.27 1.27)) hide))
-    (property "JLC" "Basic" (at 243.84 81.28 0) (effects (font (size 1.27 1.27)) hide))
+    (property "JLC" "Preferred" (at 243.84 81.28 0) (effects (font (size 1.27 1.27)) hide))
     (pin "1")
     (pin "2")
@@
     (property "Datasheet" "~" (at 365.76 83.82 0) (effects (font (size 1.27 1.27)) hide))
     (property "LCSC" "C23147" (at 365.76 83.82 0) (effects (font (size 1.27 1.27)) hide))
-    (property "JLC" "Basic" (at 365.76 83.82 0) (effects (font (size 1.27 1.27)) hide))
+    (property "JLC" "Preferred" (at 365.76 83.82 0) (effects (font (size 1.27 1.27)) hide))
     (pin "1")
     (pin "2")
@@
     (property "Datasheet" "~" (at 63.5 121.92 0) (effects (font (size 1.27 1.27)) hide))
     (property "LCSC" "C23221" (at 63.5 121.92 0) (effects (font (size 1.27 1.27)) hide))
-    (property "JLC" "Basic" (at 63.5 121.92 0) (effects (font (size 1.27 1.27)) hide))
+    (property "JLC" "Preferred" (at 63.5 121.92 0) (effects (font (size 1.27 1.27)) hide))
     (pin "1")
     (pin "2")
@@
     (property "Datasheet" "~" (at 91.44 119.38 0) (effects (font (size 1.27 1.27)) hide))
     (property "LCSC" "C4197" (at 91.44 119.38 0) (effects (font (size 1.27 1.27)) hide))
-    (property "JLC" "Basic" (at 91.44 119.38 0) (effects (font (size 1.27 1.27)) hide))
+    (property "JLC" "Preferred" (at 91.44 119.38 0) (effects (font (size 1.27 1.27)) hide))
     (pin "1")
     (pin "2")
@@
     (property "Datasheet" "~" (at 434.34 119.38 0) (effects (font (size 1.27 1.27)) hide))
     (property "LCSC" "C23265" (at 434.34 119.38 0) (effects (font (size 1.27 1.27)) hide))
-    (property "JLC" "Basic" (at 434.34 119.38 0) (effects (font (size 1.27 1.27)) hide))
-    (pin "1")
-    (pin "2")
+    (property "JLC" "Preferred" (at 434.34 119.38 0) (effects (font (size 1.27 1.27)) hide))
+    (pin "1")
+    (pin "2")
