File: hardware/kicad/lfp8_power.kicad_sch (KiCad schematic)
At the start: 21 parts, among them J1 PWR 5V, U1 AMS1117-3.3, U2 CJ431 2.495V, U3 LM358

Commit message: Firmware: one IR pulse per scan sweep; researched JLCPCB cost estimate
- fix: IR measurements that became ready together ran back to back, each
  holding the ADC ~1.1 s, so the other channels went stale and faulted
  (FAULT_ADC). The scanner now starts at most one IR pulse per full sweep,
  round robin. New regression tests: 8 simultaneous IRs, and 3 IRs while
  5 channels discharge (78 host tests pass, ESP32-C3 build OK)
- parts: 7 resistor values are JLC 'preferred extended' (no loading fee),
  not basic; labels corrected, schematic regenerated (netlist unchanged)
- ORDERING_AND_ASSEMBLY: per-board cost table for 2 / 5 / 10 assembled boards
  from fee research, the JLC part database and 2026 checkout records

Co-Authored-By: Claude Opus 5.5 <noreply@anthropic.com>
Claude-Session: https://claude.ai/code/session_01741JMFwAZptriPav2AH4Eo
Parts:
- R6, R7: JLC Basic -> Preferred
Changed lines of the file:
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@@
     (property "Datasheet" "~" (at 345.44 48.26 0) (effects (font (size 1.27 1.27)) hide))
     (property "LCSC" "C12447" (at 345.44 48.26 0) (effects (font (size 1.27 1.27)) hide))
-    (property "JLC" "Basic" (at 345.44 48.26 0) (effects (font (size 1.27 1.27)) hide))
+    (property "JLC" "Preferred" (at 345.44 48.26 0) (effects (font (size 1.27 1.27)) hide))
     (pin "1")
     (pin "2")
@@
     (property "Datasheet" "~" (at 360.68 43.18 0) (effects (font (size 1.27 1.27)) hide))
     (property "LCSC" "C23159" (at 360.68 43.18 0) (effects (font (size 1.27 1.27)) hide))
-    (property "JLC" "Basic" (at 360.68 43.18 0) (effects (font (size 1.27 1.27)) hide))
+    (property "JLC" "Preferred" (at 360.68 43.18 0) (effects (font (size 1.27 1.27)) hide))
     (pin "1")
     (pin "2")
