File: hardware/kicad/lfp8.kicad_pcb (KiCad board)
At the start: 2 copper layers, 216 x 146 mm, 835 parts, among them J1 PWR 5V, J101 XH-6P, J2 FAN 5V, J201 XH-6P, J3 USB/PROG, J301 XH-6P, J4 AUX, J401 XH-6P, J501 XH-6P, J601 XH-6P, J701 XH-6P, J801 XH-6P, Q10 BSS138, Q101 AO3401A, Q102 MMBT3904, Q103 2N7002, Q104 AO3400A, Q105 AO3400A, Q106 MMBT3904, Q107 MMBT3906, Q108 AO3400A, Q109 MMBT3906, Q11 BSS138, Q110 MMBT3904, Q111 MMBT3904, Q12 BSS138, Q13 BSS138, Q14 AO3400A, Q201 AO3401A, Q202 MMBT3904, Q203 2N7002, Q204 AO3400A, Q205 AO3400A, Q206 MMBT3904, Q207 MMBT3906, Q208 AO3400A, Q209 MMBT3906, Q210 MMBT3904, Q211 MMBT3904, Q301 AO3401A, Q302 MMBT3904, Q303 2N7002, Q304 AO3400A, Q305 AO3400A, Q306 MMBT3904, Q307 MMBT3906, Q308 AO3400A, Q309 MMBT3906, Q310 MMBT3904, Q311 MMBT3904, Q401 AO3401A, Q402 MMBT3904, Q403 2N7002, Q404 AO3400A, Q405 AO3400A, Q406 MMBT3904, Q407 MMBT3906, Q408 AO3400A, Q409 MMBT3906, Q410 MMBT3904, Q411 MMBT3904, Q501 AO3401A, Q502 MMBT3904, Q503 2N7002, Q504 AO3400A, Q505 AO3400A, Q506 MMBT3904, Q507 MMBT3906, Q508 AO3400A, Q509 MMBT3906, Q510 MMBT3904, Q511 MMBT3904, Q601 AO3401A, Q602 MMBT3904, Q603 2N7002, Q604 AO3400A, Q605 AO3400A, Q606 MMBT3904, Q607 MMBT3906, Q608 AO3400A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

Commit message: PCB: tiled routing (route one channel, replicate x8, then the common section)
Routing the whole board in one Freerouting run did not finish within 2 h.
route_tiled.py routes channel 1 alone with stub pads that bring every
off-channel net to the column's top edge, copies the result to all eight
identical channels by translation (nets renamed per channel), and leaves only
the common section for a final global pass. route_pcb.py helpers take explicit
DSN/SES paths. lfp8.kicad_pcb is the regenerated placement (corner holes),
still unrouted.

Co-Authored-By: Claude Opus 5.5 <noreply@anthropic.com>
Claude-Session: https://claude.ai/code/session_01741JMFwAZptriPav2AH4Eo
Parts:
- moved H3 45.5 mm to (34.5, 171.5)
- moved H2 29.5 mm to (241.5, 34.5)
- moved C3 23.5 mm to (33.0, 132.5)
- moved C4 23.5 mm to (37.0, 132.5)
- moved D1 18.5 mm to (35.0, 152.5)
- moved C1 11.5 mm to (33.0, 138.0)
- moved C2 11.5 mm to (37.0, 138.0)
- moved J1 6.72 mm to (35.5, 164.5)
- moved D2 2.50 mm to (35.0, 144.5)
- moved C19 1.00 mm to (202.5, 46.7)
- moved C20 1.00 mm to (206.0, 56.3)
- moved Q12 1.00 mm to (205.9, 53.2)
- moved Q13 1.00 mm to (201.4, 54.7)
- moved R40 1.00 mm to (206.5, 49.8)
- moved R42 1.00 mm to (202.3, 50.5)
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Routing:
- net +5V: track 710.9 -> 730.9 mm
